File: Starbie.kicad_sch (KiCad schematic)
At the start: 7 parts, among them SW1 SW_Push, SW2 SW_Push, U1 XIAO-ESP32-C3-SMD, U4 DHT11

Commit message: Finished the PCB, and exported.
Parts:
- U3: footprint Connector_PinHeader_2.54mm:PinHeader_1x08_P2.54mm_Vertical -> Imported Parts:MPU6050_Module
Changed lines of the file:
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@@
 			)
 		)
-		(property "Footprint" "Connector_PinHeader_2.54mm:PinHeader_1x08_P2.54mm_Vertical"
+		(property "Footprint" "Imported Parts:MPU6050_Module"
 			(at 170.18 123.19 0)
 			(hide yes)
